File: akkupack-ng.kicad_pcb (KiCad board)
At the start: 4 copper layers, 110 x 80 mm, 135 parts, among them J101 12V OUT, J102 36V IN, J103 36V OUT, J104 BAT, J105 OUT, J106 IN, J107 LED SW, J108 TEMP, J201 DISP, J202 SWD, J203 SPI, J204 USB serial, J301 USB serial, J401 USB serial, Q101 2N7002, Q102 BSS84, Q103 2N7002, Q201 2N7002, SW101 LED Enable, SW201 Reset, U101 BQ34Z100PWR-G1, U102 74HC164, U103 74HC164, U201 STM32F103CBT6, U202 USBLC6-2SC6, U203 AMS1117-3.3, U301 USBLC6-2SC6, U302 XC6206PxxxMR, U303 CH330N, U401 USBLC6-2SC6, U402 XC6206PxxxMR, U403 CH330N, Y201 8MHz, Y202 32k

Commit message: Add Blender marks
Signed-off-by: Benedikt Spranger <bene@eurovibes.org>
Other:
- board text added: "PCB3D_BR_akkupack-ng"
- board text added: "PCB3D_TL_akkupack-ng"
Changed lines of the file:
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@@
+		)
+	)
+	(gr_text "PCB3D_TL_akkupack-ng"
+		(at 50 45 180)
+		(layer "Cmts.User")
+		(effects
+			(font
+				(size 1 1)
+				(thickness 0.15)
+			)
+			(justify left bottom)
+		)
+	)
+	(gr_text "PCB3D_BR_akkupack-ng"
+		(at 160 125 0)
+		(layer "Cmts.User")
+		(effects
+			(font
+				(size 1 1)
+				(thickness 0.15)
+			)
+			(justify left bottom)
 		)
 	)
